Commit message: added IMU

File: mobility_ctrl/src/nav2_stanley/urdf/ack_rover.xacro.urdf (robot description, URDF)
Before this commit: robot ack_rover, 9 links, 8 joints
Links:
- added link imu_link, mass ${imu_mass}; collision box size=${imu_length_x} ${imu_length_y} ${imu_height}; visual box size=${imu_length_x} ${imu_length_y} ${imu_height}
Joints:
- added joint imu_joint: type fixed, parent chassis, child imu_link, origin xyz=${imu_position}

Commit message: Added GPS link and remapped /ackermann_steering/controller/tf_odometry to /tf for odom frame

File: mobility_ctrl/src/nav2_stanley/urdf/ack_rover.xacro.urdf (robot description, URDF)
Before this commit: robot ack_rover, 10 links, 9 joints
Links:
- added link gnss_link, mass 0.005; collision sphere radius=0.05; visual sphere radius=0.05
Joints:
- added joint gnss_joint: type fixed, parent chassis, child gnss_link, origin xyz=0 0 ${chassis_height} rpy=0 0 0

Commit message: Added camera function and bridge for results

File: mobility_ctrl/src/nav2_stanley/urdf/ack_rover.xacro.urdf (robot description, URDF)
Before this commit: robot ack_rover, 11 links, 10 joints
Links:
- added link camera_link; visual box size=${camera_length_x} ${camera_length_y} ${camera_height}; visual cylinder length=${camera_cyl_length} radius=${camera_cyl_radius}
- added link camera_link_optical
- link gnss_link: mass 0.005 -> ${gps_mass}; geometry collision sphere radius=${gps_radius}; visual sphere radius=${gps_radius}
Joints:
- added joint camera_joint: type fixed, parent chassis, child camera_link, origin xyz=${camera_position} rpy=0 0.18 0
- added joint camera_optical_joint: type fixed, parent camera_link, child camera_link_optical, origin xyz=0 0 0 rpy=${-pi/2} 0 ${-pi/2}
- joint gnss_joint: origin xyz=0 0 ${chassis_height} rpy=0 0 0 -> xyz=${gps_position} rpy=0 0 0

Commit message: Added inflation layers to costmap

File: mobility_ctrl/src/nav2_stanley/urdf/ack_rover.xacro.urdf (robot description, URDF)
Before this commit: robot ack_rover, 13 links, 12 joints
Joints:
- joint left_wheel_steering_joint: origin xyz=${steering_offset_x} -${wheel_offset_y} ${wheel_offset_z} rpy=${pi_div_2} 0 0 -> xyz=${steering_offset_x} ${wheel_offset_y} ${wheel_offset_z} rpy=${pi_div_2} 0 0
- joint right_wheel_steering_joint: origin xyz=${steering_offset_x} ${wheel_offset_y} ${wheel_offset_z} rpy=${pi_div_2} 0 0 -> xyz=${steering_offset_x} -${wheel_offset_y} ${wheel_offset_z} rpy=${pi_div_2} 0 0
