Commit message: Added navigation YAML for diff drive option

File: mobility_ctrl/src/nav2_stanley/urdf/diff_drive/diff_drive.xacro.urdf (robot description, URDF)
Before this commit: robot diff_drive_rover, 13 links, 12 joints
Links:
- removed link camera_link
- removed link camera_link_optical
- removed link gnss_link
- removed link imu_link
- removed link left_wheel_steering
- removed link right_wheel_steering
Joints:
- removed joint camera_joint
- removed joint camera_optical_joint
- removed joint gnss_joint
- removed joint imu_joint
- removed joint left_wheel_steering_joint
- removed joint right_wheel_steering_joint
- joint chassis_joint: origin xyz=${chassis_offset_x} ${chassis_offset_y} ${chassis_offset_z} rpy=0 0 0 -> xyz=0 0 0.5 rpy=0 0 0
- joint front_left_wheel_joint: origin xyz=0 0 0 rpy=0 0 0 -> xyz=-${wheel_offset_x} ${wheel_offset_y} ${wheel_offset_z} rpy=-${pi_div_2} 0 0; parent left_wheel_steering -> chassis
- joint front_right_wheel_joint: origin xyz=0 0 0 rpy=0 0 0 -> xyz=-${wheel_offset_x} -${wheel_offset_y} ${wheel_offset_z} rpy=-${pi_div_2} 0 0; parent right_wheel_steering -> chassis
- joint rear_left_wheel_joint: origin xyz=-${wheel_offset_x} ${wheel_offset_y} ${wheel_offset_z} rpy=-${pi_div_2} 0 0 -> xyz=${wheel_offset_x} ${wheel_offset_y} ${wheel_offset_z} rpy=-${pi_div_2} 0 0
- joint rear_right_wheel_joint: origin xyz=-${wheel_offset_x} -${wheel_offset_y} ${wheel_offset_z} rpy=-${pi_div_2} 0 0 -> xyz=${wheel_offset_x} -${wheel_offset_y} ${wheel_offset_z} rpy=-${pi_div_2} 0 0
