Commit message: jetson cubemars

File: mobility_ctrl/src/cubemars_test/urdf/cubemars.xacro.urdf (robot description, URDF)
Before this commit: robot cubemars_motor, 1 links, 1 joints
Links:
- removed link ${joint_name}_link
- added link base_link; visual box size=0.5 0.5 0.05
- added link wheel_1_link, mass 1.0; collision sphere radius=0.05; visual sphere radius=0.05
Joints:
- removed joint ${joint_name}
- added joint $wheel_1_joint: type continuous, parent base_link, child wheel_1_link, origin xyz=0.5 0.5 0 rpy=0 0 0, axis 0 0 1

File: mobility_ctrl/src/nav2_stanley/urdf/ack_rover.xacro.urdf (robot description, URDF)
Before this commit: robot ack_rover, 9 links, 8 joints
Joints:
- added joint base_to_plate: type fixed, parent zed_multi_link, child base_link, origin xyz=0 0 -0.8 rpy=0 0 0
