Commit message: Zeroing motors

File: mobility_ctrl/src/rover_hw/urdf/rover.xacro.urdf (robot description, URDF)
Before this commit: robot ack_rover, 9 links, 8 joints
Links:
- added link left_rear_steering, mass ${steering_mass}
- added link right_rear_steering, mass ${steering_mass}
Joints:
- added joint left_rear_steering_joint: type revolute, parent chassis, child right_rear_steering, origin xyz=-${steering_offset_x} ${wheel_offset_y} ${wheel_offset_z} rpy=${pi_div_2} 0 0, axis ${steering_axis}, limit lower=${steering_limit_lower} upper=${steering_limit_upper} effort=${steering_effort} velocity=${steering_velocity}
- added joint right_rear_steering_joint: type revolute, parent chassis, child right_rear_steering, origin xyz=-${steering_offset_x} -${wheel_offset_y} ${wheel_offset_z} rpy=${pi_div_2} 0 0, axis ${steering_axis}, limit lower=${steering_limit_lower} upper=${steering_limit_upper} effort=${steering_effort} velocity=${steering_velocity}

Commit message: rover_hw functioning on actual hardware. Bugs with steering angle

File: mobility_ctrl/src/rover_hw/urdf/rover.xacro.urdf (robot description, URDF)
Before this commit: robot ack_rover, 11 links, 10 joints
Links:
- removed link left_rear_steering
- removed link right_rear_steering
Joints:
- removed joint left_rear_steering_joint
- removed joint right_rear_steering_joint
- joint front_left_wheel_joint: axis ${wheel_axis} -> ${wheel_axis_left}
- joint front_right_wheel_joint: axis ${wheel_axis} -> ${wheel_axis_right}
- joint rear_left_wheel_joint: axis ${wheel_axis} -> ${wheel_axis_left}; origin xyz=-${wheel_offset_x} ${wheel_offset_y} ${wheel_offset_z} rpy=-${pi_div_2} 0 0 -> xyz=-${wheel_offset_x} ${wheel_offset_y} ${wheel_offset_z} rpy=-${pi_div_2} 0 3.14159
- joint rear_right_wheel_joint: axis ${wheel_axis} -> ${wheel_axis_right}

Commit message: Updates to rover_hw with corrected steering orientation (Added enc_off parameter)

File: mobility_ctrl/src/rover_hw/urdf/rover.xacro.urdf (robot description, URDF)
Before this commit: robot rover, 9 links, 8 joints
Joints:
- joint front_left_wheel_joint: axis ${wheel_axis_left} -> ${wheel_axis_left_front}
- joint front_right_wheel_joint: axis ${wheel_axis_right} -> ${wheel_axis_right_front}
- joint left_wheel_steering_joint: axis ${steering_axis} -> ${steering_axis_left}; origin xyz=${steering_offset_x} ${wheel_offset_y} ${wheel_offset_z} rpy=${pi_div_2} 0 0 -> xyz=${steering_offset_x} ${wheel_offset_y} ${wheel_offset_z} rpy=-${pi_div_2} 0 0
- joint rear_left_wheel_joint: axis ${wheel_axis_left} -> ${wheel_axis_left_rear}; origin xyz=-${wheel_offset_x} ${wheel_offset_y} ${wheel_offset_z} rpy=-${pi_div_2} 0 3.14159 -> xyz=-${wheel_offset_x} ${wheel_offset_y} ${wheel_offset_z} rpy=-${pi_div_2} 0 0
- joint rear_right_wheel_joint: axis ${wheel_axis_right} -> ${wheel_axis_right_rear}
- joint right_wheel_steering_joint: axis ${steering_axis} -> ${steering_axis_right}; origin xyz=${steering_offset_x} -${wheel_offset_y} ${wheel_offset_z} rpy=${pi_div_2} 0 0 -> xyz=${steering_offset_x} -${wheel_offset_y} ${wheel_offset_z} rpy=-${pi_div_2} 0 0

Commit message: Initial nav2 hardware

File: mobility_ctrl/src/rover_hw/urdf/rover.xacro.urdf (robot description, URDF)
Before this commit: robot rover, 9 links, 8 joints
Links:
- added link $(arg camera_name_0)_camera_link
- added link $(arg camera_name_1)_camera_link
- added link $(arg multi_link)
Joints:
- added joint $(arg camera_name_0)_camera_joint: type fixed, parent $(arg camera_name_0)_camera_link, child $(arg multi_link), origin xyz=-0.06 0.0 0.0 rpy=0 0 0
- added joint $(arg camera_name_1)_camera_joint: type fixed, parent $(arg multi_link), child $(arg camera_name_1)_camera_link, origin xyz=-0.06 0.0 0.0 rpy=0 0 ${M_PI}
- added joint base_link_joint: type fixed, parent $(arg camera_name_0)_camera_link, child base_link, origin xyz=0 0 -1.0 rpy=0 0 0

Commit message: Moving macro to rover URDF

File: mobility_ctrl/src/rover_hw/urdf/rover.xacro.urdf (robot description, URDF)
Before this commit: robot rover, 12 links, 11 joints
Joints:
- joint base_link_joint: origin xyz=0 0 -1.0 rpy=0 0 0 -> xyz=0.03 0 -0.4 rpy=0 0 0

Commit message: Working cameras w/ correct TF tree, map not published yet

File: mobility_ctrl/src/rover_hw/urdf/rover.xacro.urdf (robot description, URDF)
Before this commit: robot rover, 12 links, 11 joints
Links:
- removed link $(arg camera_name_0)_camera_link
- removed link $(arg camera_name_1)_camera_link
